File: board/freetronics_oled128.sch (KiCad schematic (older format))
At the start: 34 parts, among them IC1 TPS61040, P1 CONN_8

Commit message: Add MicroSD & relevant connections to schematic
Parts:
- removed P1: CONN_8, symbol CONN_8
- added C?: 100nF, symbol C
- added P?: MICROSD, symbol MICROSD
- added P?: CONN_10, symbol CONN_10
- added Q?: 2N7002, SOT23, symbol 2N7002
- added R?: 2K7, symbol R
- added R?: 1K5, symbol R
- added R?: 10K, symbol R
- added R?: 4K7, symbol R
Connections:
- net labels added: MISO, MISO_3v3, MOSI_3v3, OLED_DNC, OLED_RST, OLED_nCS, SCK_3v3, uSD_CD, uSD_nCS
- net labels removed: DNC, RST, nCS
- wire segments 113 -> 162
- no-connect marks 8 -> 7
Other:
- note added: "MicroSD Slot"
- note added: "SPI Level Shifting"
- moved on the sheet: C1, Q?, R10, R11, R13, R14, R5, R6, R8, R9, R?, REG1

Commit message: Add GPIO1 PTH
Parts:
- added JP?: GPIO1, symbol M01
Connections:
- wire segments 162 -> 138
- no-connect marks 7 -> 5

Commit message: Revert boost converter to 15V output, using values from Marc's
Inductor changed from 4.7uH to 6.8uH as I calculated a 5V input
voltage meant a 30% higher FsMax than 3.3V input, so increased the
inductor in proportion to compensate...
Parts:
- C6: value 10pF -> 22pF
- L1: value 8.2uH -> 6.8uH
- R3: value 91K 1% -> 82K 1%
Other:
- note added: "OLED VCC = 15V\nMax current draw <50mA"
- note added: "OLED VCC Supply 15V DC"
- note removed: "OLED VCC = 13.5V\nMax current draw <50mA"
- note removed: "OLED VCC Supply 13.5V DC"
Changed lines of the file:
@@
-EESchema Schematic File Version 2  date Wed 20 Feb 2013 17:22:50 EST
+EESchema Schematic File Version 2  date Wed 20 Feb 2013 17:49:20 EST
 LIBS:power
 LIBS:device
@@
 Freetronics OLED128
 Text Notes 1400 5550 0    80   ~ 0
-OLED VCC Supply 13.5V DC
+OLED VCC Supply 15V DC
 Text Notes 1400 3950 0    80   ~ 0
 3.3v Supply
@@
 $EndComp
 Text Notes 5100 6000 0    60   ~ 0
-OLED VCC = 13.5V\nMax current draw <50mA
+OLED VCC = 15V\nMax current draw <50mA
 $Comp
 L +5V #PWR05
@@
 P 4150 6250
 F 0 "C6" H 4200 6350 50  0000 L CNN
-F 1 "10pF" H 4200 6150 50  0000 L CNN
+F 1 "22pF" H 4200 6150 50  0000 L CNN
 	1    4150 6250
 	1    0    0    -1
@@
 P 3750 6750
 F 0 "R3" V 3830 6750 50  0000 C CNN
-F 1 "91K 1%" V 3650 6750 50  0000 C CNN
+F 1 "82K 1%" V 3650 6750 50  0000 C CNN
 	1    3750 6750
 	1    0    0    -1
@@
 P 2500 5800
 F 0 "L1" V 2450 5800 40  0000 C CNN
-F 1 "8.2uH" V 2600 5800 40  0000 C CNN
+F 1 "6.8uH" V 2600 5800 40  0000 C CNN
 	1    2500 5800
 	0    -1   -1   0

Commit message: Update schematic to pass ERC
Parts:
- removed P?: MICROSD, symbol MICROSD
- added P2: MICROSD, symbol MICROSD
- gave numbers to parts that had none: 11
- renumbered R4 to R10, R8 to R13, R9 to R14, R13 to R15, R14 to R16, R15 to R17, R5 to R2, R6 to R3, R10 to R5, R11 to R6, R2 to R8, R3 to R9
